Commit message: Mock-up model completed. Need to measure exact lengths.

File: urdf/mikrorobot_arm.urdf (robot description, URDF)
Before this commit: robot mikrorobot_arm, 2 links, 1 joints
Links:
- added link link_2; visual box size=0.02 0.015 0.15
- added link link_3; visual box size=0.02 0.015 0.08
- added link link_4; visual box size=0.02 0.015 0.06
Joints:
- added joint joint_2: type revolute, parent link_1, child link_2, origin xyz=0 0 0.1 rpy=0 0 0, axis 1 0 0, limit lower=-1.548 upper=1.548 effort=1000.0 velocity=0.5
- added joint joint_3: type revolute, parent link_2, child link_3, origin xyz=0 0 0.15 rpy=0 0 0, axis 1 0 0, limit lower=-1.548 upper=1.548 effort=1000.0 velocity=0.5
- added joint joint_4: type revolute, parent link_3, child link_4, origin xyz=0 0 0.08 rpy=0 0 0, axis 1 0 0, limit lower=-1.548 upper=1.548 effort=1000.0 velocity=0.5
- joint joint_1: origin xyz=0 0 0 rpy=0 0 0 -> xyz=0 0 0.025 rpy=0 0 0
